Commit message: Imprived simple bot by adding caster and sensors. Adding an emply node that should implement wall following.

File: simplebot_description/urdf/simplebot.urdf.xacro (robot description, xacro)
@@ -1,4 +1,6 @@
 <?xml version="1.0"?>
 <robot xmlns:xacro="http://www.ros.org/wiki/xacro" name="SimpleBot">
+  <!-- Include the file that contains sonar description. -->
+  <xacro:include filename="$(find hector_sensors_description)/urdf/sonar_sensor.urdf.xacro" />
   <!-- The definition of colors used in this urdf -->
   <material name="white">
@@ -134,3 +136,70 @@
     <plugin name="gazebo_ros_control" filename="libgazebo_ros_control.so" />
   </gazebo>
+  <!--Caster wheel of the robot  -->
+  <link name="caster_link">
+    <visual>
+      <origin rpy="1.0 0 0" xyz="0 0 0"/>
+      <geometry>
+        <sphere radius="0.075"/>
+      </geometry>
+      <material name="black"/>
+    </visual>
+    <collision>
+      <geometry>
+        <sphere radius="0.075"/>
+      </geometry>
+      <origin rpy="0 0 0" xyz="0 0 0"/>
+    </collision>
+    <inertial>
+      <mass value="0.5"/>
+      <origin xyz="0 0 0"/>
+      <inertia ixx="0.001" ixy="0.0" ixz="0.0" iyy="0.001" iyz="0.0" izz="0.001"/>
+    </inertial>
+  </link>
+  <joint name="caster_joint" type="fixed">
+    <parent link="base_link"/>
+    <child link="caster_link"/>
+    <origin rpy="0 0 0" xyz="-0.35 0 0"/>
+  </joint>
+  <gazebo reference="caster_link">
+    <turnGravityOff>false</turnGravityOff>
+    <mu1 value="0.0"/>
+    <mu2 value="0.0"/>
+  </gazebo>
+  <!-- Sonar sensor facing forward -->
+  <xacro:sonar_sensor
+    name="front_sonar"
+    parent="base_link"
+    ros_topic="front_sonar"
+    update_rate="10"
+    min_range="0.01"
+    max_range="5.00"
+    field_of_view="${5*pi/180}"
+    ray_count="3">
+    <origin xyz="0.35 0 0.15" rpy="0 0 0"/>
+  </xacro:sonar_sensor>
+  <!-- Sonar sensor facing to the left -->
+  <xacro:sonar_sensor
+    name="left_sonar"
+    parent="base_link"
+    ros_topic="left_sonar"
+    update_rate="10"
+    min_range="0.01"
+    max_range="5.00"
+    field_of_view="${5*pi/180}"
+    ray_count="3">
+    <origin xyz="0.35 0 0.15" rpy="0 0 ${M_PI/2}"/>
+  </xacro:sonar_sensor>
+  <!-- Sonar sensor facing to the right -->
+  <xacro:sonar_sensor
+    name="righ_sonar"
+    parent="base_link"
+    ros_topic="right_sonar"
+    update_rate="10"
+    min_range="0.01"
+    max_range="5.00"
+    field_of_view="${5*pi/180}"
+    ray_count="3">
+    <origin xyz="0.35 0 0.15" rpy="0 0 -${M_PI/2}"/>
+  </xacro:sonar_sensor>
 </robot>

Commit message: Adding package necessary for L2 completion. L2 description still work in prograss.

File: simplebot_description/urdf/simplebot.urdf.xacro (robot description, xacro)
@@ -203,3 +203,63 @@
     <origin xyz="0.35 0 0.15" rpy="0 0 -${M_PI/2}"/>
   </xacro:sonar_sensor>
+  <!-- Macro defining hokuyo lidar units -->
+  <xacro:macro name="hokuyo_lidar" params="side x y z yaw">
+    <!-- Lidar link -->
+    <link name="${side}_laser_link">
+      <collision>
+        <origin xyz="0 0 -0.0225" rpy="0 0 0"/>
+        <geometry>
+          <box size="0.05 0.05 0.07"/>
+        </geometry>
+      </collision>
+      <visual>
+        <origin xyz="0 0 -0.0225" rpy="0 0 0"/>
+        <geometry>
+          <box size="0.05 0.05 0.07"/>
+        </geometry>
+        <material name="white"/>
+      </visual>
+    </link>
+    <!-- Joint connecting lidar to base_link -->
+    <joint name="${side}_laser_joint" type="fixed">
+      <parent link="base_link"/>
+      <child link="${side}_laser_link"/>
+      <origin xyz="${x} ${y} ${z}" rpy="0 0 ${yaw}"/>
+    </joint>
+    <!-- Gazebo tag describing how the lidar is simulated in Gazebo -->
+    <gazebo reference="${side}_laser_link">
+      <sensor name="${side}_laser" type="ray">
+        <pose>0 0 0 0 0 0</pose>
+        <ray>
+          <scan>
+            <horizontal>
+              <!-- The URG-04LX-UG01  has  683 steps with 0.35139 Degree resolution -->
+              <resolution>1</resolution>
+              <max_angle>2.0944</max_angle>
+              <!-- 120 Degree -->
+              <min_angle>-2.0944</min_angle>
+              <!-- -120 Degree -->
+              <samples>683</samples>
+            </horizontal>
+          </scan>
+          <range>
+            <min>0.2</min>
+            <max>20</max>
+            <resolution>0.01</resolution>
+          </range>
+        </ray>
+        <plugin name="${side}_laser" filename="libgazebo_ros_laser.so">
+          <topicName>${side}_laser/${side}_scan</topicName>
+          <frameName>${side}_laser_link</frameName>
+        </plugin>
+        <always_on>1</always_on>
+        <update_rate>10</update_rate>
+        <!-- You can change this property to true to visualize lidar rays in Gazebo -->
+        <visualize>false</visualize>
+      </sensor>
+    </gazebo>
+  </xacro:macro>
+  <!-- Now we actually create two lidar instances that are added to our robot -->
+  <xacro:hokuyo_lidar side="front" x="0.35" y="0" z="0.15" yaw="0"/>
+  <xacro:hokuyo_lidar side="back" x="-0.35" y="0" z="0.15" yaw="${M_PI}"/>
 </robot>

Commit message: Adding IMU sensor to simplebot description file.

File: simplebot_description/urdf/simplebot.urdf.xacro (robot description, xacro)
@@ -263,3 +263,32 @@
   <xacro:hokuyo_lidar side="front" x="0.35" y="0" z="0.15" yaw="0"/>
   <xacro:hokuyo_lidar side="back" x="-0.35" y="0" z="0.15" yaw="${M_PI}"/>
+  <!-- Here we create necessary links and joints of IMU device -->
+  <link name="imu_link"/>
+  <joint name="imu_joint" type="fixed">
+    <parent link="base_link"/>
+    <child link="imu_link"/>
+    <origin xyz="0.0 0.0 0.0" rpy="0 0 0"/>
+  </joint>
+  <gazebo>
+    <!-- Plugin that simulates IMU device in Gazebo -->
+    <plugin name="imu_sim" filename="libhector_gazebo_ros_imu.so">
+      <serviceName>/imu/calibrate</serviceName>
+      <updateRate>200.0</updateRate>
+      <bodyName>imu_link</bodyName>
+      <frameId>imu_link</frameId>
+      <topicName>imu_data</topicName>
+      <rpyOffset>0 0 0</rpyOffset>
+      <xyzOffset>0 0 0</xyzOffset>
+      <gaussianNoise>0.00000001</gaussianNoise>
+      <accelDrift>0.00000001 0.00000001 0.00000001</accelDrift>
+      <accelDriftFrequency>0.00000001 0.00000001 0.00000001</accelDriftFrequency>
+      <accelGaussianNoise>0.00000001 0.00000001 0.00000001</accelGaussianNoise>
+      <rateDrift>0.0 0.0 0.0</rateDrift>
+      <rateDriftFrequency>0.0 0.0 0.0</rateDriftFrequency>
+      <rateGaussianNoise>0.0 0.0 0.0</rateGaussianNoise>
+      <headingDrift>0.0 0.0 0.0</headingDrift>
+      <headingDriftFrequency>0.0 0.0 0.0</headingDriftFrequency>
+      <headingGaussianNoise>0.0 0.0 0.0</headingGaussianNoise>
+    </plugin>
+  </gazebo>
 </robot>
